File: hardware/easyeda_pcb_to_kicad/espip_boy_rev2.kicad_sch (KiCad schematic)
At the start: 112 parts, among them CN1 1X4, P2 CONN_01X04, Q1 SS8050/Y1, Q2 SS8050/Y1, Q3 DMG1012T-7, Q4 DMG1012T-7, Q5 SS8050/Y1, SW1 TS24CA 250GF 013, SW4 TS24CA 250GF 013, U1 LTR-390UV-01, U10 ICS-43434_C5656610, U11 ME6217A33PG, U12 BQ24074RGTR, U13 MAX30102EFD+T_C6454833, U14 BQ27421YZFR-G1A, U15 200_mah_lipo, U17 MAX98357AETE+T, U18 ME6206B18XG, U2 CP2102N-A02-GQFN28R, U3 0402 Blue, U4 GT-USB-7010ASV, U5 BMI270, U6 1.69"_Display, U7 YSN8010SJ 32.768KHZ, U8 ESP32-WROOM-32E(8MB), U9 LIS2MDLTR

Commit message: Completed assembly of Rev 2 pcb, battery, display and digital crown
Parts:
- LED1, U3: footprint (none) -> LED_SMD:LED_0402_1005Metric
- SW1: footprint (none) -> easyeda2kicad:SW-SMD_L4.7-W3.5-P3.35-EH
- U2: footprint Package_DFN_QFN:QFN-28-1EP_5x5mm_P0.5mm_EP2.7x2.7mm -> Package_DFN_QFN:QFN-28-1EP_5x5mm_P0.5mm_EP3.35x3.35mm_ThermalVias
Changed lines of the file:
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@@
 		(lib_id "TS24CA 250GF 013")
 		(at 138.43 144.78 0)
-		(unit 0)
+		(unit 1)
 		(exclude_from_sim no)
 		(in_bom yes)
@@
 			)
 		)
-		(property "Footprint" ""
+		(property "Footprint" "easyeda2kicad:SW-SMD_L4.7-W3.5-P3.35-EH"
 			(at 138.43 144.78 0)
 			(effects
@@
 				(path "/b3258cd7-0bc0-483d-8fcd-4f864f109cc4"
 					(reference "SW1")
-					(unit 0)
+					(unit 1)
 				)
 			)
@@
 			)
 		)
-		(property "Footprint" "Package_DFN_QFN:QFN-28-1EP_5x5mm_P0.5mm_EP2.7x2.7mm"
+		(property "Footprint" "Package_DFN_QFN:QFN-28-1EP_5x5mm_P0.5mm_EP3.35x3.35mm_ThermalVias"
 			(at 205.74 83.82 0)
 			(effects
@@
 		(lib_id "XL-1005UBC_C22355736")
 		(at 320.04 80.01 0)
-		(unit 0)
+		(unit 1)
 		(exclude_from_sim no)
 		(in_bom yes)
@@
 			)
 		)
-		(property "Footprint" ""
+		(property "Footprint" "LED_SMD:LED_0402_1005Metric"
 			(at 320.04 80.01 0)
 			(effects
@@
 				(path "/b3258cd7-0bc0-483d-8fcd-4f864f109cc4"
 					(reference "U3")
-					(unit 0)
+					(unit 1)
 				)
 			)
@@
 		(lib_id "TZ-P2-0402YGTIA1-0.45T")
 		(at 320.04 85.09 0)
-		(unit 0)
+		(unit 1)
 		(exclude_from_sim no)
 		(in_bom yes)
@@
 			)
 		)
-		(property "Footprint" ""
+		(property "Footprint" "LED_SMD:LED_0402_1005Metric"
 			(at 320.04 85.09 0)
 			(effects
@@
 				(path "/b3258cd7-0bc0-483d-8fcd-4f864f109cc4"
 					(reference "LED1")
-					(unit 0)
+					(unit 1)
 				)
 			)
